File: DESAIN PCB/FLIGHT_CONTROLLER/FLIGHT_CONTROLLER.kicad_pcb (KiCad board)
At the start: 2 copper layers, 82.9 x 83.1 mm, 63 parts, among them J1 POWER CONNECTOR, J10 ESC INPUT, J11 ESC INPUT, J12 RC TRANSMITTER, J13 TRANSMITTER, J14 GY-88A, J15 FTDI BREAKOUT BOARD, J16 ESC POWER, J2 SPI PROG, J3 USB B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

Commit message: [board] complete
Connections:
- J3 pad 5: unconnected-(J3-Pad5) -> (no net)
Other:
- board text added: "82.931 mm"
- board text added: "83.058 mm"

Commit message: [board] correction
Parts:
- removed kibuzzard-63E0D02C: G***, kibuzzard-63E0D02C
- removed kibuzzard-63E0D05B: G***, kibuzzard-63E0D05B
- added kibuzzard-63E733C3: G***, kibuzzard-63E733C3, B.Cu at (149.1, 142.2)
- added kibuzzard-63E7341A: G***, kibuzzard-63E7341A, B.Cu at (134.6, 142.2)
- added kibuzzard-63E7348F: G***, kibuzzard-63E7348F, F.Cu at (141.2, 102.9)
- added kibuzzard-63E734BE: G***, kibuzzard-63E734BE, B.Cu at (179.1, 102.9)
- moved J1 7.20 mm to (138.2, 136.9), turned to 180 degrees
Connections:
- J1 pad 1: Net-(F1-Pad1) -> GND
- J1 pad 2: GND -> Net-(F1-Pad1)
Other:
- board text removed: "82.931 mm"
- board text removed: "83.058 mm"

Commit message: add PCB V.1.2
Parts:
- C14: value 0.1uF -> DNP
Connections:
- J3 pad 5: (no net) -> unconnected-(J3-Pad5)
Changed lines of the file:
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@@
   (net 58 "unconnected-(J15-Pad1)")
   (net 59 "unconnected-(J15-Pad5)")
+  (net 60 "unconnected-(J3-Pad5)")
   (footprint "Connector_PinSocket_2.54mm:PinSocket_1x06_P2.54mm_Vertical" (layer "F.Cu")
     (at 162.56 85.09 -90)
@@
       (net 1 "GND") (pinfunction "GND") (pintype "power_out"))
     (pad "5" thru_hole circle (at 4.86 7.25 180) (size 4 4) (drill 2.3) (layers *.Cu *.Mask)
-      (pinfunction "Shield") (pintype "passive"))
+      (net 60 "unconnected-(J3-Pad5)") (pinfunction "Shield") (pintype "passive"))
     (pad "5" thru_hole circle (at 4.86 -4.75 180) (size 4 4) (drill 2.3) (layers *.Cu *.Mask)
-      (pinfunction "Shield") (pintype "passive"))
+      (net 60 "unconnected-(J3-Pad5)") (pinfunction "Shield") (pintype "passive"))
     (model "${KIPRJMOD}/LIBRARY/3D MODEL LIBRARY/USB TYPEB.STEP"
       (offset (xyz 7 -1.2 0))
@@
     (attr board_only exclude_from_pos_files exclude_from_bom)
     (fp_text reference "kibuzzard-63E7348F" (at 0 -4.869077 -90) (layer "F.SilkS") hide
-      (effects (font (size 0 0)))
+      (effects (font (size 0 0) (thickness 0.15)))
     )
     (fp_text value "G***" (at 0 4.869077 -90) (layer "F.SilkS") hide
-      (effects (font (size 0 0)))
+      (effects (font (size 0 0) (thickness 0.15)))
     )
     (fp_poly (pts
@@
     (attr board_only exclude_from_pos_files exclude_from_bom)
     (fp_text reference "kibuzzard-63E7341A" (at 0 4.531114) (layer "B.SilkS") hide
-      (effects (font (size 0 0)) (justify mirror))
+      (effects (font (size 0 0) (thickness 0.15)) (justify mirror))
     )
     (fp_text value "G***" (at 0 -4.531114) (layer "B.SilkS") hide
-      (effects (font (size 0 0)) (justify mirror))
+      (effects (font (size 0 0) (thickness 0.15)) (justify mirror))
     )
     (fp_poly (pts
@@
     (attr board_only exclude_from_pos_files exclude_from_bom)
     (fp_text reference "kibuzzard-63E733C3" (at 0 4.531114) (layer "B.SilkS") hide
-      (effects (font (size 0 0)) (justify mirror))
+      (effects (font (size 0 0) (thickness 0.15)) (justify mirror))
     )
     (fp_text value "G***" (at 0 -4.531114) (layer "B.SilkS") hide
-      (effects (font (size 0 0)) (justify mirror))
+      (effects (font (size 0 0) (thickness 0.15)) (justify mirror))
     )
     (fp_poly (pts
@@
     (property "Sheetname" "")
     (attr smd)
-    (fp_text reference "C3" (at 3.048 0 90) (layer "B.SilkS")
+    (fp_text reference "C3" (at 3.048 -0.762 90) (layer "B.SilkS")
       (effects (font (size 1 1) (thickness 0.15)) (justify mirror))
     )
@@
       (effects (font (size 1 1) (thickness 0.15)) (justify mirror))
     )
-    (fp_text value "0.1uF" (at 0 -1.68) (layer "B.Fab")
+    (fp_text value "DNP" (at 0 -1.68) (layer "B.Fab")
       (effects (font (size 1 1) (thickness 0.15)) (justify mirror))
     )
@@
     (property "Sheetname" "")
     (attr smd)
-    (fp_text reference "C1" (at 0 1.68 90) (layer "B.SilkS")
+    (fp_text reference "C1" (at -0.762 1.68 90) (layer "B.SilkS")
       (effects (font (size 1 1) (thickness 0.15)) (justify mirror))
     )
@@
     (attr board_only exclude_from_pos_files exclude_from_bom)
     (fp_text reference "kibuzzard-63E734BE" (at 0 4.869077 90) (layer "B.SilkS") hide
-      (effects (font (size 0 0)) (justify mirror))
+      (effects (font (size 0 0) (thickness 0.15)) (justify mirror))
     )
     (fp_text value "G***" (at 0 -4.869077 90) (layer "B.SilkS") hide
-      (effects (font (size 0 0)) (justify mirror))
+      (effects (font (size 0 0) (thickness 0.15)) (justify mirror))
     )
     (fp_poly (pts
@@
     (property "Sheetname" "")
     (attr smd)
-    (fp_text reference "C6" (at 3.048 0 90) (layer "B.SilkS")
+    (fp_text reference "C6" (at 3.048 0.762 90) (layer "B.SilkS")
       (effects (font (size 1 1) (thickness 0.15)) (justify mirror))
     )
