File: DESAIN PCB/FLIGHT_CONTROLLER/FLIGHT_CONTROLLER.kicad_sch (KiCad schematic)
At the start: 49 parts, among them J1 POWER CONNECTOR, J10 ESC INPUT, J11 ESC INPUT, J12 RC TRANSMITTER, J13 TRANSMITTER, J14 GY-88A, J15 FTDI BREAKOUT BOARD, J16 ESC POWER, J2 SPI PROG, J3 USB B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

Commit message: add PCB V.1.2
Parts:
- C14: value 0.1uF -> DNP
Other:
- note added: "AUX2 = D8"
Changed lines of the file:
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@@
     (effects (font (size 1.27 1.27)) (justify left bottom))
+  )
+  (text "AUX2 = D8" (at 215.646 100.838 0)
+    (effects (font (size 1 1)) (justify left bottom))
   )
   (text "DECOUPLING CAPACITOR" (at 132.08 66.04 0)
@@
     (in_bom yes) (on_board yes)
     (property "Reference" "C14" (id 0) (at 170.815 26.67 90))
-    (property "Value" "0.1uF" (id 1) (at 170.815 28.575 90))
+    (property "Value" "DNP" (id 1) (at 170.815 28.575 90))
     (property "Footprint" "Capacitor_SMD:C_0805_2012Metric_Pad1.18x1.45mm_HandSolder" (id 2) (at 170.815 31.75 0)
       (effects (font (size 1.27 1.27)) hide)
@@
     )
     (path "/b2f9dbed-d299-494a-bfb3-262becf62c80"
-      (reference "C14") (unit 1) (value "0.1uF") (footprint "Capacitor_SMD:C_0805_2012Metric_Pad1.18x1.45mm_HandSolder")
+      (reference "C14") (unit 1) (value "DNP") (footprint "Capacitor_SMD:C_0805_2012Metric_Pad1.18x1.45mm_HandSolder")
     )
     (path "/d46f6994-a34c-434d-bc59-13723b0819f7"
