File: DESAIN PCB/FLIGHT_CONTROLLER_REV_2/FLIGHT_CONTROLLER_REV_2.kicad_pcb (KiCad board)
At the start: 2 copper layers, 46 parts, among them J1 AVR-ISP-10, J10 GPS INPUT, J11 AVR-ISP-10, J2 USB B, J3 Conn_01x03_Male, J4 Conn_01x03_Male, J5 Conn_01x03_Male, J6 Conn_01x03_Male, J7 Conn_01x08_Female, J8 Conn_01x08_Female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

Commit message: add PCB REV 2
Parts:
- added H1: MountingHole, MountingHole:MountingHole_3.2mm_M3_ISO7380_Pad, F.Cu at (76.2, 138.4)
- added H2: MountingHole, MountingHole:MountingHole_3.2mm_M3_ISO7380_Pad, F.Cu at (147.3, 47.0)
- added H3: MountingHole, MountingHole:MountingHole_3.2mm_M3_ISO7380_Pad, F.Cu at (76.2, 47.0)
- added H4: MountingHole, MountingHole:MountingHole_3.2mm_M3_ISO7380_Pad, F.Cu at (147.3, 138.4)
- added J12: TRANSMITTER_1, Connector_PinHeader_2.54mm:PinHeader_1x04_P2.54mm_Vertical, F.Cu at (89.2, 81.3)
- added J13: TRANSMITTER_2, Connector_PinHeader_2.54mm:PinHeader_1x04_P2.54mm_Vertical, F.Cu at (89.2, 77.5)
- added R10: 1K, Resistor_THT:R_Axial_DIN0207_L6.3mm_D2.5mm_P7.62mm_Horizontal, F.Cu at (135.6, 72.6)
- added R11: 1K, Resistor_THT:R_Axial_DIN0207_L6.3mm_D2.5mm_P7.62mm_Horizontal, F.Cu at (131.6, 72.6)
- U2: moved to B.Cu
- moved J3 218.1 mm to (89.7, 133.8), turned to 180 degrees
- moved J5 209.7 mm to (85.9, 133.8), turned to 180 degrees
- moved J11 206.0 mm to (138.5, 130.2), turned to 180 degrees
- moved J6 205.9 mm to (93.5, 133.9), turned to 180 degrees
- moved C1 204.5 mm to (91.4, 118.0)
- moved J1 197.6 mm to (114.3, 129.5), turned to -90 degrees
- moved R2 197.0 mm to (123.2, 127.0), turned to -90 degrees
- moved J7 196.8 mm to (82.0, 120.5), turned to 180 degrees
- moved D1 193.9 mm to (128.3, 129.5), turned to -90 degrees
- moved Y2 192.6 mm to (126.7, 102.8), turned to 90 degrees
- moved J4 187.3 mm to (82.0, 133.8), turned to 180 degrees
- moved C6 180.2 mm to (125.4, 109.2)
- moved D5 178.2 mm to (128.3, 126.2), turned to 90 degrees
- moved J8 177.6 mm to (116.0, 105.4), turned to 180 degrees
- moved C8 176.0 mm to (125.4, 91.4)
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Connections:
- J1 pad 1: /MAIN_CONTROLLER/MOSI -> /MAIN_CONTROLLER/D11
- U1 pad 17: /MAIN_CONTROLLER/MOSI -> /MAIN_CONTROLLER/D11
- U3 pad 2: /GPS/RX -> Net-(U3-Pad2)
- U3 pad 3: /GPS/TX -> Net-(U3-Pad3)
Routing:
- net +5V: track 0.00 -> 573.9 mm, vias 0 -> 14
- net GND: track 0.00 -> 480.8 mm, vias 0 -> 14
- net /MAIN_CONTROLLER/RST: track 0.00 -> 126.7 mm, vias 0 -> 6
- net /GPS/RST: track 0.00 -> 116.3 mm, vias 0 -> 4
- net SDA: track 0.00 -> 72.7 mm
- net SCL: track 0.00 -> 69.5 mm
- net /MAIN_CONTROLLER/RX_LED: track 0.00 -> 60.5 mm
- net /MAIN_CONTROLLER/SCK: track 0.00 -> 57.4 mm, vias 0 -> 2
- net /MAIN_CONTROLLER/TX_LED: track 0.00 -> 54.9 mm
- net /MAIN_CONTROLLER/D11: track 0.00 -> 54.4 mm, vias 0 -> 2
- net /MAIN_CONTROLLER/D3: track 0.00 -> 50.0 mm, vias 0 -> 2
- net /GPS/SCK: track 0.00 -> 40.6 mm, vias 0 -> 2
- net /MAIN_CONTROLLER/D4: track 0.00 -> 36.0 mm
- net /MAIN_CONTROLLER/TX: track 0.00 -> 34.9 mm
- net /MAIN_CONTROLLER/D2: track 0.00 -> 33.2 mm
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- added copper zone on B.Cu, net GND
Other:
- board outline added: 78.7 x 99.1 mm
