File: DESAIN PCB/FLIGHT_CONTROLLER_REV_2/GPS.kicad_sch (KiCad schematic)
At the start: 15 parts, among them J10 GPS INPUT, J11 AVR-ISP-10, J9 FTDI BREAKOUT BOARD, SW2 SW_SPST, U3 ATmega328P-P, Y2 16 MHz

Commit message: add PCB REV 2
Parts:
- added R10, R11: 1K, Resistor_THT:R_Axial_DIN0207_L6.3mm_D2.5mm_P7.62mm_Horizontal, symbol Device:R_Small
Connections:
- net RX: now also R10.2; no longer U3.2 (PD0)
- net TX: now also R11.2; no longer U3.3 (PD1)
- new net: R10.1, U3.2 (PD0)
- new net: R11.1, U3.3 (PD1)
Changed lines of the file:
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@@
+    (stroke (width 0) (type default) (color 0 0 0 0))
+  )
+  (wire (pts (xy 78.486 81.534) (xy 82.296 81.534))
     (stroke (width 0) (type default) (color 0 0 0 0))
   )
@@
     (stroke (width 0) (type default) (color 0 0 0 0))
   )
+  (wire (pts (xy 78.486 78.994) (xy 82.296 78.994))
+    (stroke (width 0) (type default) (color 0 0 0 0))
+  )
   (wire (pts (xy 29.718 117.221) (xy 29.718 117.856))
     (stroke (width 0) (type default) (color 0 0 0 0))
@@
     (stroke (width 0) (type default) (color 0 0 0 0))
   )
-  (wire (pts (xy 73.406 78.994) (xy 82.296 78.994))
-    (stroke (width 0) (type default) (color 0 0 0 0))
-  )
   (wire (pts (xy 116.078 56.134) (xy 116.078 56.388))
     (stroke (width 0) (type default) (color 0 0 0 0))
@@
   )
   (polyline (pts (xy 18.034 59.69) (xy 18.034 56.134))
-    (stroke (width 0) (type default) (color 0 0 0 0))
-  )
-  (wire (pts (xy 73.406 81.534) (xy 82.296 81.534))
     (stroke (width 0) (type default) (color 0 0 0 0))
   )
@@
     (pin "2")
   )
+  (symbol (lib_id "Device:R_Small") (at 75.946 78.994 90) (unit 1)
+    (in_bom yes) (on_board yes)
+    (property "Reference" "R10" (id 0) (at 76.2 77.216 90))
+    (property "Value" "1K" (id 1) (at 75.946 78.994 90))
+    (property "Footprint" "Resistor_THT:R_Axial_DIN0207_L6.3mm_D2.5mm_P7.62mm_Horizontal" (id 2) (at 75.946 78.994 0)
+      (effects (font (size 1.27 1.27)) hide)
+    )
+    (property "Datasheet" "~" (id 3) (at 75.946 78.994 0)
+      (effects (font (size 1.27 1.27)) hide)
+    )
+    (pin "1")
+    (pin "2")
+  )
   (symbol (lib_id "power:GND") (at 29.21 83.566 90) (unit 1)
     (in_bom yes) (on_board yes)
@@
       (effects (font (size 1.27 1.27)) hide)
     )
+    (pin "1")
+    (pin "2")
+  )
+  (symbol (lib_id "Device:R_Small") (at 75.946 81.534 90) (unit 1)
+    (in_bom yes) (on_board yes)
+    (property "Reference" "R11" (id 0) (at 76.2 83.312 90))
+    (property "Value" "1K" (id 1) (at 75.946 81.534 90))
+    (property "Footprint" "Resistor_THT:R_Axial_DIN0207_L6.3mm_D2.5mm_P7.62mm_Horizontal" (id 2) (at 75.946 81.534 0)
+      (effects (font (size 1.27 1.27)) hide)
+    )
+    (property "Datasheet" "~" (id 3) (at 75.946 81.534 0)
+      (effects (font (size 1.27 1.27)) hide)
+    )
